File: premierProjet/premierProjet.kicad_pcb (KiCad board)
At the start: 2 copper layers, 13 parts, among them J1 Conn_01x02_Male, SW1 Push, SW2 Push, SW3 Push, SW4 Push

Commit message: PCB Complet pour premier projet
YOLO
Routing:
- net /Masse: track 74.5 -> 0.00 mm
- net /Plus: track 56.0 -> 71.1 mm
- added copper zone on F.Cu, net /Masse
Other:
- board outline added: 53.8 x 28.4 mm
