File: Sharp G850-Interface/Sharp G850-Interface.kicad_pcb (KiCad board)
At the start: 2 copper layers, 53.3 x 36.6 mm, 28 parts, among them J1 USB_B_Micro, J2 Conn_01x11_Male, J3 Conn_01x11_Male, U1 FT232RL

Commit message: Finished PCB + Added gerber files
Parts:
- J2: footprint Connector_PinHeader_2.54mm:PinHeader_1x11_P2.54mm_Horizontal -> hwreverse:PinHeader_1x11_G850
Connections:
- J2 pad 1: (no net) -> FG
- J2 pad 10: (no net) -> DSRCalc
- J2 pad 11: (no net) -> CICalc
- J2 pad 2: (no net) -> VCCCalc
- J2 pad 5: (no net) -> DTRCalc
- J2 pad 8: (no net) -> CDCalc
- J3 pad 1: (no net) -> FG
- J3 pad 10: (no net) -> DSRCalc
- J3 pad 11: (no net) -> CICalc
- J3 pad 2: (no net) -> VCCCalc
- J3 pad 5: (no net) -> DTRCalc
- J3 pad 8: (no net) -> CDCalc
Routing:
- net (no net): track 24.4 -> 0.00 mm
- net VCCCalc: track 0.00 -> 4.06 mm
- net FG: track 0.00 -> 4.06 mm
- net DTRCalc: track 0.00 -> 4.06 mm
- net DSRCalc: track 0.00 -> 4.06 mm
- net CICalc: track 0.00 -> 4.06 mm
- net CDCalc: track 0.00 -> 4.06 mm
- net GND: vias 10 -> 42
Other:
- board text added: "+RX"
- board text added: "+TX"
- board text added: "3V3"
- board text added: "5V"
- board text added: "Interface USB pour Sharp PC-G850"
- board text added: "PWR+"
- board text added: "VCC-I/O"
- board text added: "https://www.twitch.tv/alexx_and_seb"
