File: MD-100 Emulator/MD-100 Emulator.sch (KiCad schematic (older format))
At the start: 48 parts, among them J1 CPB_Connector, J2 I2CConn, J3 ICSP, Q1 NPN, U1 24LC1025, U2 24LC1025, U3 24LC1025, U4 24LC1025, U5 74HC00, U6 74HC02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

Commit message: Routage du PCB MD-100 terminé
Parts:
- U1, U2, U3, U4: footprint Package_SO:SOIC-8-1EP_3.9x4.9mm_P1.27mm_EP2.29x3mm -> Package_SO:SOIC-8_3.9x4.9mm_P1.27mm
Connections:
- net GND: now also J2.1 (Pin_1); no longer J2.4 (Pin_4)
- net SCL: now also J2.2 (Pin_2); no longer J2.3 (Pin_3)
- net SDA: now also J2.3 (Pin_3); no longer J2.2 (Pin_2)
- net VCC: now also J2.4 (Pin_4); no longer C2.1, C8.1, J2.1 (Pin_1)
- net VDD: now also C2.1, C8.1
- net EE1D: now reaches R1.2, U1.5 (SDA)
- net EE1C: now reaches R2.2, U1.6 (SCL)
- net EE2D: now reaches R3.2, U2.5 (SDA)
- net EE2C: now reaches R4.2, U2.6 (SCL)
- net EE3D: now reaches R5.2, U3.5 (SDA)
- net EE3C: now reaches R6.2, U3.6 (SCL)
- net EE4D: now reaches R7.2, U4.5 (SDA)
- net EE4C: now reaches R8.2, U4.6 (SCL)
- net uCC: now reaches R13.2, U7.37 (SCK/SCL/RC3)
- net uCD: now reaches R11.2, U7.42 (SDI/SDA/RC4)
