File: Toile/Toile.sch (KiCad schematic (older format))
At the start: 0 parts

Commit message: Cours du 22.06.2020
Changed lines of the file:
@@
+	1    0    0    -1
+$EndComp
+$Comp
+L porcschema:LOGO #G?
+U 1 1 5EF10E7B
+P 2500 4300
+F 0 "#G?" H 2500 3815 60  0001 C CNN
+F 1 "LOGO" H 2500 4785 60  0001 C CNN
+F 2 "" H 2500 4300 50  0001 C CNN
+F 3 "" H 2500 4300 50  0001 C CNN
+	1    2500 4300
+	1    0    0    -1
+$EndComp
+$Comp
+L porcschema2:LOGO #G?
+U 1 1 5EF1E2B1
+P 3850 4350
+F 0 "#G?" H 3850 4195 60  0001 C CNN
+F 1 "LOGO" H 3850 4505 60  0001 C CNN
+F 2 "" H 3850 4350 50  0001 C CNN
+F 3 "" H 3850 4350 50  0001 C CNN
+	1    3850 4350
 	1    0    0    -1
 $EndComp
