File: Carte Son Arduino-Mega/Carte Son Arduino-Mega.sch (KiCad schematic (older format))
At the start: 18 parts, among them J1 AudioJack3, U1 CPCB_YM2413B, U2 LMC660, Y1 Crystal

Commit message: debut cours n°18
Parts:
- added XA?: Arduino_Mega2560_Shield, symbol arduino:Arduino_Mega2560_Shield
Other:
- moved on the sheet: C1, C2, C3, C4, C5, C6, C7, J1, L1, R1, R2, R3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

Commit message: carte son opll cours final
Parts:
- added J1, J10, J11, J12, J13, J14, J17, J2, J3, J5, J7, J9: SolidPad-Connector, Connector:SolidPad_4x4mm_2x2mmCore, symbol hwreverse:SolidPad-Connector
- added J15, J8: Conn_01x08_Male, Connector_PinHeader_2.54mm:PinHeader_1x08_P2.54mm_Vertical, symbol Connector:Conn_01x08_Male
- added J16, J6: Conn_01x04_Male, Connector_PinHeader_2.54mm:PinHeader_1x04_P2.54mm_Vertical, symbol Connector:Conn_01x04_Male
- C1: renamed from C6; value C_Small -> 10uF; footprint (none) -> Capacitor_SMD:C_0805_2012Metric_Pad1.15x1.40mm_HandSolder
- C2: renamed from C5; value C_Small -> 15nF; footprint (none) -> Capacitor_SMD:C_0805_2012Metric_Pad1.15x1.40mm_HandSolder
- C3: renamed from C1; value C_Small -> 15pF; footprint (none) -> Capacitor_SMD:C_0805_2012Metric_Pad1.15x1.40mm_HandSolder
- C4: renamed from C7; value C_Small -> 10uF; footprint (none) -> Capacitor_SMD:C_0805_2012Metric_Pad1.15x1.40mm_HandSolder
- C5: renamed from C2; value C_Small -> 15pF; footprint (none) -> Capacitor_SMD:C_0805_2012Metric_Pad1.15x1.40mm_HandSolder
- C6: renamed from C3; value CP -> 1000uF; footprint (none) -> Capacitor_SMD:CP_Elec_10x12.6
- C7: renamed from C4; value C_Small -> 100nF; footprint (none) -> Capacitor_SMD:C_0805_2012Metric_Pad1.15x1.40mm_HandSolder
- J4: renamed from J1; footprint (none) -> hwreverse:BOOMELE_PJ-320B
- L1: value L -> 1mH; footprint (none) -> Inductor_SMD:L_0805_2012Metric_Pad1.15x1.40mm_HandSolder
- R1: renamed from R5; value R_Small -> 2k2; footprint (none) -> Resistor_SMD:R_0805_2012Metric_Pad1.15x1.40mm_HandSolder
- R2: renamed from R3; footprint (none) -> Resistor_SMD:R_0805_2012Metric_Pad1.15x1.40mm_HandSolder
- R3: renamed from R4; footprint (none) -> Resistor_SMD:R_0805_2012Metric_Pad1.15x1.40mm_HandSolder
- R4: renamed from R6; value R_Small -> 4k7; footprint (none) -> Resistor_SMD:R_0805_2012Metric_Pad1.15x1.40mm_HandSolder
- R5: renamed from R1; value R_Small -> 10k; footprint (none) -> Resistor_SMD:R_0805_2012Metric_Pad1.15x1.40mm_HandSolder
- R6: renamed from R2; value R_Small -> 4k7; footprint (none) -> Resistor_SMD:R_0805_2012Metric_Pad1.15x1.40mm_HandSolder
- U2: renamed from U1; footprint (none) -> Package_DIP:DIP-18_W7.62mm_Socket
- XA1: renamed from XA?; footprint (none) -> Arduino:Arduino_Mega2560_Shield
- Y1: value Crystal -> 3.57MHz; footprint (none) -> Crystal:Crystal_SMD_HC49-SD_HandSoldering
- renumbered U2 to U1
Connections:
- net GND: now also XA1.GND5 (GND), XA1.GND6 (GND), J17.~, J6.1 (Pin_1), J6.2 (Pin_2), J6.3 (Pin_3), J6.4 (Pin_4), J8.1 (Pin_1), J8.2 (Pin_2), J8.3 (Pin_3), J8.4 (Pin_4), J8.5 (Pin_5), J8.6 (Pin_6), J8.7 (Pin_7), J8.8 (Pin_8), J9.~
- net VCC: now also XA1.5V3 (5V), XA1.5V4 (5V), J14.~
- net VREG: now also U1.12, J7.~; no longer U1.3
- net A0: now reaches U2.10 (A0)
- net A0: now also XA1.A0, J13.~, J16.1 (Pin_1)
- net ~WE: now reaches U2.11 (~WE)
- net ~WE: now also XA1.A3, J10.~, J16.4 (Pin_4)
- net ~CS: now reaches U2.12 (~CS)
- net ~CS: now also XA1.A1, J12.~, J16.2 (Pin_2)
- net ~IC: now reaches U2.13 (~IC)
- net ~IC: now also XA1.A2, J11.~, J16.3 (Pin_3)
- net D0: now reaches U2.17 (D0)
- net D0: now also XA1.A8, J15.1 (Pin_1)
- net D1: now reaches U2.18 (D1)
- net D1: now also XA1.A9, J15.2 (Pin_2)
- net D2: now reaches U2.2 (D2)
- net D2: now also XA1.A10, J15.3 (Pin_3)
- net D3: now reaches U2.3 (D3)
- net D3: now also XA1.A11, J15.4 (Pin_4)
- net D4: now reaches U2.4 (D4)
- net D4: now also XA1.A12, J15.5 (Pin_5)
- net D5: now reaches U2.5 (D5)
- net D5: now also XA1.A13, J15.6 (Pin_6)
- net D6: now reaches U2.6 (D6)
- net D6: now also XA1.A14, J15.7 (Pin_7)
- net D7: now reaches U2.7 (D7)
- net D7: now also XA1.A15, J15.8 (Pin_8)
- net at R1.2, R2.1, R3.1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: now also J1.~
- net at C2.2, R4.1, U1.9: now also U1.3, J2.~; no longer U1.12
- net at C4.2, J4.R: now also J5.~
- net at C1.2, J4.T: now also J3.~
- new net: U1.13, U1.14, U1.5
- new net: C1.1, U1.1, U1.2
- no-connect marks 0 -> 75
